File: PTP_Adrian_Pavlovic_Project1/PTP_Adrian_Pavlovic_Project1.kicad_pcb (KiCad board)
At the start: 2 copper layers, 45 parts, among them J1 Screw_Terminal_01x02, SW1 SW_Push, SW2 SW_SPDT_312, U1 LM2574N-5, U2 4027, U3 4027, U4 74LS47, U5 HDSP-7401, U6 74LVC1G11, U7 NE555P

Commit message: LV8
Parts:
- moved R20 85.5 mm to (86.0, 128.0), turned to -90 degrees
- moved R19 85.5 mm to (86.0, 121.2), turned to -90 degrees
- moved U7 81.4 mm to (89.4, 119.7)
- moved U5 80.8 mm to (166.8, 110.2)
- moved R6 79.2 mm to (160.8, 121.2), turned to 0 degrees
- moved R5 78.7 mm to (160.7, 118.6), turned to 0 degrees
- moved R8 57.2 mm to (161.0, 125.2)
- moved R7 38.0 mm to (134.2, 133.8), turned to 90 degrees
- moved R9 36.9 mm to (137.5, 133.8), turned to 90 degrees
- moved R10 34.6 mm to (140.8, 133.8), turned to 90 degrees
- moved R13 34.5 mm to (130.8, 133.8), turned to 90 degrees
- moved U6 32.6 mm to (111.9, 118.0), turned to 180 degrees
- moved R11 29.7 mm to (144.0, 134.0), turned to 90 degrees
- moved R1 26.3 mm to (151.2, 84.6)
- moved C4 26.2 mm to (93.2, 131.0), turned to 180 degrees
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Routing:
- net +5V: track 0.00 -> 88.8 mm, vias 0 -> 3
- net Q0: track 0.00 -> 61.0 mm
- net GND: track 0.00 -> 59.8 mm
- net Clock: track 0.00 -> 54.4 mm, vias 0 -> 2
- net Q1: track 0.00 -> 52.3 mm, vias 0 -> 4
- net Q3: track 0.00 -> 51.0 mm, vias 0 -> 1
- net Reset: track 0.00 -> 45.4 mm, vias 0 -> 4
- net Net-(U7-THR): track 0.00 -> 33.8 mm, vias 0 -> 2
- net Net-(SW2-A): track 0.00 -> 31.5 mm
- net Q2: track 0.00 -> 24.4 mm
- net 555: track 0.00 -> 23.8 mm
- net Net-(U2A-J): track 0.00 -> 22.2 mm, vias 0 -> 2
- net VD: track 0.00 -> 21.4 mm
- net Net-(U5-B): track 0.00 -> 17.9 mm, vias 0 -> 2
- net Net-(U3A-J): track 0.00 -> 17.2 mm
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- added copper zone on B.Cu, net GND

Commit message: LV9
Routing:
- net +5V: track 88.8 -> 218.1 mm, vias 3 -> 14
- net Net-(U4-BI): track 0.00 -> 29.3 mm, vias 0 -> 2
- net Net-(D4-K): track 0.00 -> 27.5 mm
- net Q3: track 51.0 -> 62.9 mm
- net Net-(U7-DIS): track 15.4 -> 24.5 mm, vias 0 -> 2
- net Q2: track 24.4 -> 32.7 mm, vias 0 -> 2
- net Net-(U3B-J): track 12.8 -> 20.9 mm, vias 0 -> 2
- net Net-(R13-Pad1): track 4.59 -> 11.1 mm
- net Net-(U7-THR): track 33.8 -> 30.2 mm
- net Net-(U3A-J): track 17.2 -> 19.7 mm
- net Net-(U2A-J): track 22.2 -> 24.8 mm
- net Net-(U2B-J): track 16.7 -> 19.2 mm
Other:
- board outline added: 100 x 80 mm
- board text added: "PTP - BCD counter Adrian Pavlović"
